Commit message: moved simulation to ignition gazebo

File: robot/description/dept_camera.xacro (robot description, xacro)
@@ -25,31 +25,25 @@
     </joint>
     <link name="camera_link_optical"></link>
-    <!-- Gazebo plugin for the depth camera -->
-    <gazebo reference="camera_link">
-        <!-- Material definition for Gazebo -->
-        <material>Gazebo/Red</material>
-        <sensor name="camera" type="depth">
-            <pose>0 0 0 0 0 0</pose>
-            <visualize>true</visualize>
-            <update_rate>10</update_rate>
-            <camera>
-                <horizontal_fov>1.089</horizontal_fov>
-                <image>
-                    <format>B8G8R8</format>
-                    <width>640</width>
-                    <height>480</height>
-                </image>
-                <clip>
-                    <near>0.05</near>
-                    <far>8.0</far>
-                </clip>
-            </camera>
-            <!-- Camera controller plugin -->
-            <plugin name="camera_controller" filename="libgazebo_ros_camera.so">
-                <frame_name>camera_link_optical</frame_name>
-                <min_depth>0.1</min_depth>
-                <max_depth>100.0</max_depth>
-            </plugin>
-        </sensor>
+    <gazebo reference="camera_link_optical">
+      <sensor name="depth_camera" type="depth">
+        <ignition_frame_id>camera_link_optical</ignition_frame_id>
+        <camera>
+            <horizontal_fov>1.089</horizontal_fov>
+            <image>
+                <format>B8G8R8</format>
+                <width>640</width>
+                <height>480</height>
+            </image>
+            <clip>
+                <near>0.05</near>
+                <far>8.0</far>
+            </clip>
+        </camera>
+        <always_on>1</always_on>
+        <update_rate>10</update_rate>
+        <visualize>true</visualize>
+        <topic>camera</topic>
+        <enable_metrics>true</enable_metrics>
+      </sensor>
     </gazebo>
 </robot>

File: robot/description/gazebo_controller.xacro (robot description, xacro)
@@ -1,23 +1,29 @@
 <?xml version="1.0"?>
 <robot xmlns:xacro="http://www.ros.org/wiki/xacro">
-   <!-- Two Differential-drive plugin  -->
-    <gazebo>
-        <plugin name="diff_drive_robot_plugin" filename="libgazebo_ros_diff_drive.so">
-            <!-- Wheel Information -->
-            <left_joint>left_wheel_joint</left_joint>
-            <right_joint>right_wheel_joint</right_joint>
-            <wheel_separation>0.297</wheel_separation>
-            <wheel_diameter>0.066</wheel_diameter>
-            <!-- Limits -->
-            <max_wheel_torque>200</max_wheel_torque>
-            <max_wheel_acceleration>10.0</max_wheel_acceleration>
-            <!-- Output -->
-            <!-- <odometryTopic>/odom</odometryTopic> -->
-            <odometry_frame>odom</odometry_frame>
-            <robot_base_frame>base_link</robot_base_frame>
-            <publish_odom>true</publish_odom>
-            <publish_odom_tf>true</publish_odom_tf>
-            <publish_wheel_tf>true</publish_wheel_tf>
-        </plugin>
-    </gazebo>
+  <ros2_control name="IgnitionSystem" type="system">
+    <hardware>
+      <plugin>ign_ros2_control/IgnitionSystem</plugin>
+    </hardware>
+    <joint name="left_wheel_joint">
+      <command_interface name="velocity">
+          <param name="min">-10.0</param>
+          <param name="max">10.0</param>
+      </command_interface>
+      <state_interface name="position"/>
+      <state_interface name="velocity"/>
+    </joint>
+    <joint name="right_wheel_joint">
+      <command_interface name="velocity">
+          <param name="min">-10.0</param>
+          <param name="max">10.0</param>
+      </command_interface>
+      <state_interface name="position"/>
+      <state_interface name="velocity"/>
+    </joint>
+  </ros2_control>
+  <gazebo>
+    <plugin filename="ign_ros2_control-system" name="ign_ros2_control::IgnitionROS2ControlPlugin">
+      <parameters>$(find robot)/config/diff_drive_controller.yaml</parameters>
+    </plugin>
+  </gazebo>
 </robot>

File: robot/description/lidar_sensor.xacro (robot description, xacro)
@@ -13,5 +13,7 @@
                 <cylinder radius="0.05" length="0.04"/>
             </geometry>
-            <material name="black"/>
+            <material name="black">
+                <color rgba="0 0 0 1"/>
+            </material>
         </visual>
         <visual>
@@ -20,5 +22,7 @@
                 <cylinder radius="0.01" length="0.1"/>
             </geometry>
-            <material name="black"/>
+            <material name="black">
+                <color rgba="0 0 0 1"/>
+            </material>
         </visual>
         <collision>
@@ -32,38 +36,27 @@
         </xacro:inertial_cylinder>
     </link>
-    <!-- Gazebo settings -->
     <gazebo reference="laser_frame">
-        <material>Gazebo/Blue</material> <!-- Use only one material -->
-    </gazebo>
-    <!-- LIDAR SENSOR CONFIGURATION -->
-    <gazebo reference="laser_frame">
-        <sensor name="lidar_sensor" type="ray">
-            <pose>0 0 0 0 0 0</pose>
-            <visualize>true</visualize>
-            <update_rate>40</update_rate>
-            <ray>
-                <scan>
-                    <horizontal>
-                        <samples>360</samples>
-                        <min_angle>-3.14</min_angle>
-                        <max_angle>3.14</max_angle>
-                    </horizontal>
-                </scan>
-                <range>
-                    <min>0.3</min>
-                    <max>12</max>
-                    <resolution>0.2</resolution>
-                </range>
-            </ray>
-            <!-- Updated plugin for ROS 2 -->
-            <plugin name="laser_controller" filename="libgazebo_ros_ray_sensor.so">
-                <ros>
-                    <!-- Fixed remapping syntax -->
-                    <argument>~/out:=scan</argument>
-                </ros>
-                <output_type>sensor_msgs/LaserScan</output_type>
-                <frame_name>laser_frame</frame_name>
-            </plugin>
-        </sensor>
+      <sensor name="lidar_sensor" type="gpu_lidar">
+        <pose> 0 0 0 0 0 0 </pose>
+        <ignition_frame_id>laser_frame</ignition_frame_id>
+        <topic>scan</topic>
+        <always_on>true</always_on>
+        <visualize>true</visualize>
+        <update_rate>30</update_rate>
+        <ray>
+          <scan>
+              <horizontal>
+                  <samples>360</samples>
+                  <min_angle>${-pi*2}</min_angle>
+                  <max_angle>${pi*2}</max_angle>
+              </horizontal>
+          </scan>
+          <range>
+              <min>0.3</min>
+              <max>12.0</max>
+              <resolution>0.2</resolution>
+          </range>
+        </ray>
+      </sensor>
     </gazebo>
 </robot>

File: robot/description/robot.urdf.xacro (robot description, xacro)
@@ -7,4 +7,6 @@
   <!-- The lidar sensor file  -->
   <xacro:include filename="lidar_sensor.xacro"/>
+  <!-- The imu sensor file  -->
+  <xacro:include filename="imu_sensor.xacro"/>
   <!-- dept camra file  -->
   <xacro:include filename="dept_camera.xacro"/>

File: robot/description/robot.xacro (robot description, xacro)
@@ -21,5 +21,5 @@
         <parent link="base_link"/>
         <child link="chassis"/>
-        <origin xyz="-0.1 0 0"/>
+        <origin xyz="-0.1 0 0.05"/>
     </joint>
     <link name="chassis">
@@ -29,5 +29,7 @@
                 <cylinder radius="0.3" length="0.1"/> <!-- Circular chassis -->
             </geometry>
-            <material name="blue"/>
+            <material name="blue">
+                <color rgba="0.2 0.2 1 1"/>
+            </material>
         </visual>
         <collision>
@@ -38,16 +40,12 @@
         </collision>
         <xacro:inertial_cylinder mass="0.5" radius="0.3" length="0.15">
-            <origin xyz="0.15 0 0.075" rpy="0 0 0"/>
+            <origin xyz="0.3 0 0.075" rpy="0 0 0"/>
         </xacro:inertial_cylinder>
     </link>
-    <!-- Adding colour to chassis link -->
-    <gazebo reference="chassis">
-        <material>Gazebo/Blue</material>
-    </gazebo>
     <!-- LEFT WHEEL OF ROBOT -->
     <joint name="left_wheel_joint" type="continuous">
         <parent link="base_link"/>
         <child link="left_wheel"/>
-        <origin xyz="0 0.175 0" rpy="-${pi/2} 0 0"/>
+        <origin xyz="0 0.175 0.05" rpy="-${pi/2} 0 0"/>
         <axis xyz="0 0 1"/>
     </joint>
@@ -57,5 +55,7 @@
                 <cylinder radius="0.05" length="0.04"/>
             </geometry>
-            <material name="black"/>
+            <material name="black">
+                <color rgba="0 0 0 1"/>
+            </material>
         </visual>
         <collision>
@@ -69,5 +69,6 @@
     </link>
     <gazebo reference="left_wheel">
-        <material>Gazebo/Black</material>
+        <mu1>1.0</mu1>
+        <mu2>1.0</mu2>
     </gazebo>
     <!-- RIGHT WHEEL OF ROBOT -->
@@ -75,5 +76,5 @@
         <parent link="base_link"/>
         <child link="right_wheel"/>
-        <origin xyz="0 -0.175 0" rpy="${pi/2} 0 0"/>
+        <origin xyz="0 -0.175 0.05" rpy="${pi/2} 0 0"/>
         <axis xyz="0 0 -1"/>
     </joint>
@@ -83,5 +84,7 @@
                 <cylinder radius="0.05" length="0.04"/>
             </geometry>
-            <material name="black"/>
+            <material name="black">
+                <color rgba="0 0 0 1"/>
+            </material>
         </visual>
         <collision>
@@ -95,5 +98,6 @@
     </link>
     <gazebo reference="right_wheel">
-        <material>Gazebo/Black</material>
+        <mu1>1.0</mu1>
+        <mu2>1.0</mu2>
     </gazebo>
     <!-- DOLLY WHEEL JOINT -->
@@ -101,5 +105,5 @@
         <parent link="chassis"/>
         <child link="dolly_wheel"/>
-        <origin xyz="0.24 0 0"/>
+        <origin xyz="0.34 0 0"/>
     </joint>
     <link name="dolly_wheel">
@@ -108,5 +112,7 @@
                 <sphere radius="0.05"/>
             </geometry>
-            <material name="black"/>
+            <material name="black">
+                <color rgba="0 0 0 1"/>
+            </material>
         </visual>
         <collision>
@@ -120,7 +126,6 @@
     </link>
     <gazebo reference="dolly_wheel">
-        <material>Gazebo/Black</material>
-        <mu1 value="0.100"/>
-        <mu2 value="0.100"/>
+        <mu1 value="0.001"/>
+        <mu2 value="0.001"/>
     </gazebo>
 </robot>
