Commit message: repositioned depth camera

File: zed_bot_description/urdf/controllers/epmc_diff_drive_ros2_control.xacro (robot description, xacro)
@@ -6,5 +6,5 @@
         <param name="motorA_wheel_name">left_wheel_joint</param>
         <param name="motorB_wheel_name">right_wheel_joint</param>
-        <param name="port">/dev/serial/by-path/platform-fd500000.pcie-pci-0000:01:00.0-usb-0:1.2.4:1.0-port0</param>
+        <param name="port">/dev/ttyUSB0</param>
         <param name="cmd_vel_timeout_ms">2000</param>
       </hardware>

File: zed_bot_description/urdf/dept_camera.xacro (robot description, xacro)
@@ -6,5 +6,5 @@
       <child link="camera_link"/>
       <!-- Camera origin adjusted to be at the center of the chassis -->
-      <origin xyz="0.15 -0.3 0.12" rpy="0 0 0"/> <!-- Position camera at chassis center -->
+      <origin xyz="0.45 0.0 0.15" rpy="0 0 0"/> <!-- Position camera at chassis center -->
    </joint>
     <!-- Camera link definition -->
@@ -13,5 +13,5 @@
             <geometry>
                 <!-- Changing to box for rectangular camera -->
-                <box size="0.03 0.03 0.03"/> <!-- Adjust dimensions as needed -->
+                <box size="0.03 0.12 0.03"/> <!-- Adjust dimensions as needed -->
             </geometry>
             <!-- Removed material definition here, using Gazebo plugin material instead -->
@@ -26,7 +26,7 @@
     <link name="camera_link_optical"></link>
     <xacro:if value="$(arg run_gz_sim)">
-        <gazebo reference="camera_link">
+        <gazebo reference="camera_link_optical">
           <visual>
-            <xacro:gz_material_grey/>
+            <xacro:gz_material_red/>
           </visual>
           <sensor name="camera_link_optical" type="depth">
